Commit message: Hacks with prop mesh for ABV

File: uuv_gazebo_plugins/uuv_gazebo_ros_plugins/urdf/thruster_snippets.xacro (robot description, xacro)
@@ -87,7 +87,7 @@
       </xacro:box_inertial>
       <visual>
-        <origin rpy="0 0 0" xyz="0 0 0"/>
+        <origin rpy="0 3.14159 0" xyz="-0.08 0 0.0"/>
         <geometry>
-          <mesh filename="${mesh_filename}" scale="1 1 1"/>
+          <mesh filename="${mesh_filename}" scale="0.45 0.45 0.45"/>
         </geometry>
       </visual>

Commit message: Added arguments for thruster spin axis

File: uuv_gazebo_plugins/uuv_gazebo_ros_plugins/urdf/thruster_snippets.xacro (robot description, xacro)
@@ -72,4 +72,7 @@
     params="namespace
             thruster_id
+            x_axis:=1
+            y_axis:=0
+            z_axis:=0
             *origin
             mesh_filename
@@ -78,5 +81,5 @@
     <joint name="${namespace}/thruster_${thruster_id}_joint" type="continuous">
       <xacro:insert_block name="origin"/>
-      <axis xyz="1 0 0"/>
+      <axis xyz="${x_axis} ${y_axis} ${z_axis}"/>
       <parent link="${namespace}/base_link"/>
       <child link="${namespace}/thruster_${thruster_id}"/>
@@ -122,4 +125,7 @@
       params="namespace
               thruster_id
+              x_axis:=1
+              y_axis:=0
+              z_axis:=0
               *origin
               mesh_filename
@@ -127,4 +133,7 @@
               rotor_constant">
     <xacro:generic_thruster_macro
+      x_axis="${x_axis}"
+      y_axis="${y_axis}"
+      z_axis="${z_axis}"
       namespace="${namespace}"
       thruster_id="${thruster_id}"
