Commit message: Initial Commit

File: uuv_descriptions/urdf/rexrov.gazebo.xacro (robot description, xacro)
@@ -35,5 +35,5 @@
                 <!-- Added mass: see p.28 in Berg2012 -->
                 <added_mass>
-                     779.79 -6.8773 -103.32  8.5426 -165.54 -7.8033
+                    79.79 -6.8773 -103.32  8.5426 -165.54 -7.8033
                     -6.8773    1222   51.29  409.44 -5.8488  62.726
                     -103.32   51.29  3659.9  6.1112 -386.42  10.774

File: uuv_descriptions/urdf/rexrov_sensors.xacro (robot description, xacro)
@@ -38,5 +38,5 @@
   </xacro:default_imu_macro>
   <!-- Mount a camera -->
-  <xacro:default_camera namespace="${namespace}" parent_link="${namespace}/base_link" suffix="">
+  <xacro:default_camera namespace="${namespace}" parent_link="${namespace}/base_link" suffix="depth">
     <origin xyz="1.15 0 0.4" rpy="0 0.6 0"/>
   </xacro:default_camera>

File: uuv_gazebo_plugins/uuv_gazebo_ros_plugins/urdf/thruster_snippets.xacro (robot description, xacro)
@@ -106,4 +106,6 @@
         <jointName>${namespace}/thruster_${thruster_id}_joint</jointName>
         <thrusterID>${thruster_id}</thrusterID>
+        <thrustMin>0</thrustMin>
+        <thrustMax>51.48</thrustMax>
         <xacro:insert_block name="dynamics"/>
         <xacro:insert_block name="conversion"/>
@@ -111,4 +113,107 @@
     </gazebo>
     <gazebo reference="${namespace}/thruster_${thruster_id}">
+      <selfCollide>false</selfCollide>
+    </gazebo>
+    <joint name="${namespace}/thrusterdummy_${thruster_id}_joint" type="fixed">
+      <xacro:insert_block name="origin"/>
+      <axis xyz="1 0 0"/>
+      <parent link="${namespace}/base_link"/>
+      <child link="${namespace}/thrusterdummy_${thruster_id}"/>
+    </joint>
+    <link name="${namespace}/thrusterdummy_${thruster_id}">
+      <xacro:box_inertial x="0" y="0" z="0" mass="0.001">
+        <origin xyz="0 0 0" rpy="0 0 0"/>
+      </xacro:box_inertial>
+      <visual>
+        <origin rpy="0 0 0" xyz="0 0 0"/>
+        <geometry>
+          <mesh filename="${mesh_filename}" scale="1 1 1"/>
+        </geometry>
+      </visual>
+      <collision>
+        <!-- todo: gazebo needs a collision volume or it will ignore the pose of
+           the joint that leads to this link (and assume it to be the identity) -->
+        <geometry>
+          <cylinder length="0.000001" radius="0.000001"/>
+        </geometry>
+        <origin xyz="0 0 0" rpy="0 0 0"/>
+      </collision>
+    </link>
+    <gazebo reference="${namespace}/thrusterdummy_${thruster_id}">
+      <selfCollide>false</selfCollide>
+    </gazebo>
+  </xacro:macro>
+  <xacro:macro name="bluerov2_thruster_macro"
+    params="namespace
+            thruster_id
+            *origin
+            mesh_filename
+            *dynamics
+            *conversion">
+    <joint name="${namespace}/thruster_${thruster_id}_joint" type="continuous">
+      <xacro:insert_block name="origin"/>
+      <axis xyz="1 0 0"/>
+      <parent link="${namespace}/base_link"/>
+      <child link="${namespace}/thruster_${thruster_id}"/>
+    </joint>
+    <link name="${namespace}/thruster_${thruster_id}">
+      <xacro:box_inertial x="0" y="0" z="0" mass="0.001">
+        <origin xyz="0 0 0" rpy="0 0 0"/>
+      </xacro:box_inertial>
+      <visual>
+        <origin rpy="0 0 0" xyz="0 0 0"/>
+        <geometry>
+          <mesh filename="${mesh_filename}" scale="1 1 1"/>
+        </geometry>
+      </visual>
+      <collision>
+        <!-- todo: gazebo needs a collision volume or it will ignore the pose of
+           the joint that leads to this link (and assume it to be the identity) -->
+        <geometry>
+          <cylinder length="0.000001" radius="0.000001"/>
+        </geometry>
+        <origin xyz="0 0 0" rpy="0 0 0"/>
+      </collision>
+    </link>
+    <gazebo>
+      <plugin name="${namespace}_${thruster_id}_thruster_model" filename="libuuv_thruster_ros_plugin.so">
+        <linkName>${namespace}/thruster_${thruster_id}</linkName>
+        <jointName>${namespace}/thruster_${thruster_id}_joint</jointName>
+        <thrusterID>${thruster_id}</thrusterID>
+        <thrustMin>0</thrustMin>
+        <thrustMax>51.48</thrustMax>
+        <xacro:insert_block name="dynamics"/>
+        <xacro:insert_block name="conversion"/>
+      </plugin>
+    </gazebo>
+    <gazebo reference="${namespace}/thruster_${thruster_id}">
+      <selfCollide>false</selfCollide>
+    </gazebo>
+    <joint name="${namespace}/thrusterdummy_${thruster_id}_joint" type="fixed">
+      <xacro:insert_block name="origin"/>
+      <axis xyz="1 0 0"/>
+      <parent link="${namespace}/base_link"/>
+      <child link="${namespace}/thrusterdummy_${thruster_id}"/>
+    </joint>
+    <link name="${namespace}/thrusterdummy_${thruster_id}">
+      <xacro:box_inertial x="0" y="0" z="0" mass="0.001">
+        <origin xyz="0 0 0" rpy="0 0 0"/>
+      </xacro:box_inertial>
+      <visual>
+        <origin rpy="0 0 0" xyz="0 0 0"/>
+        <geometry>
+          <mesh filename="${mesh_filename}" scale="1 1 1"/>
+        </geometry>
+      </visual>
+      <collision>
+        <!-- todo: gazebo needs a collision volume or it will ignore the pose of
+           the joint that leads to this link (and assume it to be the identity) -->
+        <geometry>
+          <cylinder length="0.000001" radius="0.000001"/>
+        </geometry>
+        <origin xyz="0 0 0" rpy="0 0 0"/>
+      </collision>
+    </link>
+    <gazebo reference="${namespace}/thrusterdummy_${thruster_id}">
       <selfCollide>false</selfCollide>
     </gazebo>
@@ -135,3 +240,19 @@
     </xacro:generic_thruster_macro>
   </xacro:macro>
+  <xacro:macro name="thruster_module_first_order_basic_fcn_macro_bluerov2"
+      params="namespace
+              thruster_id
+              *origin
+              mesh_filename
+              dyn_time_constant
+              rotor_constant">
+    <xacro:bluerov2_thruster_macro
+      namespace="${namespace}"
+      thruster_id="${thruster_id}"
+      mesh_filename="${mesh_filename}">
+      <xacro:insert_block name="origin"/>
+      <xacro:rotor_dyn_first_order_macro time_constant="${dyn_time_constant}"/>
+      <xacro:thruster_cf_basic_macro rotor_constant="${rotor_constant}"/>
+    </xacro:bluerov2_thruster_macro>
+  </xacro:macro>
 </robot>

File: uuv_sensor_plugins/uuv_sensor_ros_plugins/urdf/camera_snippets.xacro (robot description, xacro)
@@ -28,4 +28,21 @@
       parent_link="${parent_link}"
       topic="camera"
+      mass="0.001"
+      update_rate="30"
+      hfov="1.5125"
+      width="768"
+      height="492"
+      stddev="0.02"
+      scale=".50">
+      <inertia ixx="0.00001" ixy="0.0" ixz="0.0" iyy="0.00001" iyz="0.0" izz="0.00001" />
+      <xacro:insert_block name="origin" />
+    </xacro:regular_camera_plugin_macro>
+  </xacro:macro>
+  <xacro:macro name="depth_camera" params="namespace parent_link suffix *origin">
+    <xacro:depth_camera_plugin_macro
+      namespace="${namespace}"
+      suffix="${suffix}"
+      parent_link="${parent_link}"
+      topic="camera"
       mass="0.1"
       update_rate="30"
@@ -37,5 +54,5 @@
       <inertia ixx="0.00001" ixy="0.0" ixz="0.0" iyy="0.00001" iyz="0.0" izz="0.00001" />
       <xacro:insert_block name="origin" />
-    </xacro:regular_camera_plugin_macro>
+    </xacro:depth_camera_plugin_macro>
   </xacro:macro>
   <xacro:macro name="wideangle_camera" params="namespace parent_link suffix *origin">
@@ -122,7 +139,8 @@
         </camera>
         <plugin name="camera${suffix}_controller" filename="libgazebo_ros_camera.so">
+        <!-- <plugin name="camera${suffix}_controller" filename="libgazebo_ros_openni_kinect.so"> -->
           <updateRate>${update_rate}</updateRate>
           <cameraName>${namespace}/camera${suffix}</cameraName>
-          <frameName>camera${suffix}_link_optical</frameName>
+          <frameName>${namespace}/camera${suffix}_link_optical</frameName>
           <attenuationR>0.0</attenuationR>
           <attenuationG>0.0</attenuationG>
@@ -137,4 +155,98 @@
           <depthImageCameraInfoTopicName>${topic}_depth_info</depthImageCameraInfoTopicName>
           <pointCloudCutoff>10.0</pointCloudCutoff>
+        </plugin>
+      </sensor>
+    </gazebo>
+  </xacro:macro>
+  <xacro:macro name="depth_camera_plugin_macro"
+    params="namespace suffix parent_link topic mass update_rate
+      hfov width height stddev scale
+      *inertia *origin">
+    <!-- Sensor link -->
+    <link name="${namespace}/camera${suffix}_link">
+      <inertial>
+        <xacro:insert_block name="inertia" />
+        <mass value="${mass}" />
+        <origin xyz="0 0 0" rpy="0 0 0" />
+      </inertial>
+      <visual>
+        <geometry>
+          <mesh filename="file://$(find uuv_sensor_ros_plugins)/meshes/oe14-372.dae" scale="${scale} ${scale} ${scale}"/>
+        </geometry>
+      </visual>
+      <xacro:no_collision/>
+    </link>
+    <joint name="${namespace}/camera${suffix}_joint" type="revolute">
+      <xacro:insert_block name="origin" />
+      <parent link="${parent_link}" />
+      <child link="${namespace}/camera${suffix}_link" />
+      <limit upper="0" lower="0" effort="0" velocity="0" />
+      <axis xyz="1 0 0"/>
+    </joint>
+    <link name="${namespace}/camera${suffix}_link_optical">
+      <xacro:box_inertial x="0.0001" y="0.0001" z="0.0001" mass="0.001">
+        <origin xyz="0 0 0" rpy="0 0 0"/>
+      </xacro:box_inertial>
+      <collision>
+        <!-- todo: gazebo needs a collision volume or it will ignore the pose of
+           the joint that leads to this link (and assume it to be the identity) -->
+        <geometry>
+          <cylinder length="0.000001" radius="0.000001"/>
+        </geometry>
+        <origin xyz="0 0 0" rpy="0 ${0.5*pi} 0"/>
+      </collision>
+    </link>
+    <joint name="${namespace}/camera${suffix}_optical_joint" type="revolute">
+      <origin xyz="0 0 0" rpy="${-pi/2} 0 ${-pi/2}"/>
+      <parent link="${namespace}/camera${suffix}_link"/>
+      <child link="${namespace}/camera${suffix}_link_optical"/>
+      <limit upper="0" lower="0" effort="0" velocity="0" />
+      <axis xyz="1 0 0"/>
+    </joint>
+    <gazebo reference="${namespace}/camera${suffix}_link">
+      <sensor type="camera" name="camera${suffix}">
+        <update_rate>${update_rate}</update_rate>
+        <camera name="camera${suffix}">
+          <horizontal_fov>${hfov}</horizontal_fov>
+          <image>
+            <width>${width}</width>
+            <height>${height}</height>
+            <format>R8G8B8</format>
+          </image>
+          <clip>
+            <near>0.05</near>
+            <far>3000</far>
+          </clip>
+          <noise>
+            <type>gaussian</type>
+            <mean>0.0</mean>
+            <stddev>${stddev}</stddev>
+          </noise>
+        </camera>
+        <plugin name="camera${suffix}_plugin" filename="libgazebo_ros_openni_kinect.so">
+          <baseline>0.2</baseline>
+          <alwaysOn>true</alwaysOn>
+          <!-- Keep this zero, update_rate in the parent <sensor> tag
+            will control the frame rate. -->
+          <updateRate>0.0</updateRate>
+          <cameraName>camera_ir</cameraName>
+          <imageTopicName>/camera/color/image_raw</imageTopicName>
+          <cameraInfoTopicName>/camera/color/camera_info</cameraInfoTopicName>
+          <depthImageTopicName>/camera/depth/image_raw</depthImageTopicName>
+          <depthImageCameraInfoTopicName>/camera/depth/camera_info</depthImageCameraInfoTopicName>
+          <pointCloudTopicName>/camera/depth/points</pointCloudTopicName>
+          <frameName>camera_link</frameName>
+          <pointCloudCutoff>0.5</pointCloudCutoff>
+          <pointCloudCutoffMax>3.0</pointCloudCutoffMax>
+          <distortionK1>0</distortionK1>
+          <distortionK2>0</distortionK2>
+          <distortionK3>0</distortionK3>
+          <distortionT1>0</distortionT1>
+          <distortionT2>0</distortionT2>
+          <CxPrime>0</CxPrime>
+          <Cx>0</Cx>
+          <Cy>0</Cy>
+          <focalLength>0</focalLength>
+          <hackBaseline>0</hackBaseline>
         </plugin>
       </sensor>
@@ -207,4 +319,5 @@
         </camera>
         <plugin name="camera${suffix}_controller" filename="libuuv_gazebo_ros_camera_plugin.so">
+        <!-- <plugin name="camera${suffix}_controller" filename="libgazebo_ros_openni_kinect.so"> -->
           <updateRate>${update_rate}</updateRate>
           <cameraName>${namespace}/camera${suffix}</cameraName>

File: uuv_sensor_plugins/uuv_sensor_ros_plugins/urdf/imu_snippets.xacro (robot description, xacro)
@@ -93,5 +93,5 @@
       imu_suffix=""
       parent_link="${parent_link}"
-      imu_topic="imu"
+      imu_topic="imu2"
       mass_imu_sensor="0.015"
       gyroscope_noise_density="0.0003394"
