Commit message: 9-21 update

File: uuv_descriptions/urdf/rexrov_sensors.xacro (robot description, xacro)
@@ -23,7 +23,7 @@
   <xacro:default_magnetometer namespace="${namespace}" parent_link="${namespace}/base_link"/>
   <!-- RPT  -->
-  <xacro:default_rpt namespace="${namespace}" parent_link="${namespace}/base_link">
+  <!--<xacro:default_rpt namespace="${namespace}" parent_link="${namespace}/base_link">
     <origin xyz="-1.32 0 0.8" rpy="0 0 0"/>
-  </xacro:default_rpt>
+  </xacro:default_rpt>-->
   <!-- Pressure  -->
   <xacro:default_pressure_macro namespace="${namespace}" parent_link="${namespace}/base_link">

File: uuv_gazebo_plugins/uuv_gazebo_ros_plugins/urdf/thruster_snippets.xacro (robot description, xacro)
@@ -106,5 +106,5 @@
         <jointName>${namespace}/thruster_${thruster_id}_joint</jointName>
         <thrusterID>${thruster_id}</thrusterID>
-        <thrustMin>0</thrustMin>
+        <thrustMin>-51.48</thrustMin>
         <thrustMax>51.48</thrustMax>
         <xacro:insert_block name="dynamics"/>

File: uuv_sensor_plugins/uuv_sensor_ros_plugins/urdf/imu_snippets.xacro (robot description, xacro)
@@ -30,4 +30,21 @@
       imu_topic="imu"
       mass_imu_sensor="0.015"
+      gyroscope_noise_density="0.000003394"
+      gyroscope_random_walk="0.00000038785"
+      gyroscope_bias_correlation_time="100.0"
+      gyroscope_turn_on_bias_sigma="0.0087"
+      accelerometer_noise_density="0.00004"
+      accelerometer_random_walk="0.00006"
+      accelerometer_bias_correlation_time="100.0"
+      accelerometer_turn_on_bias_sigma="0.1960"
+      orientation_noise="0.00001"
+      enable_local_ned_frame="false"
+      reference_frame="world"
+      update_rate="50">
+      <inertia ixx="0.00001" ixy="0.0" ixz="0.0" iyy="0.00001" iyz="0.0" izz="0.00001" />
+      <xacro:insert_block name="origin" />
+    </xacro:imu_plugin_macro>
+  </xacro:macro>
+<!--
       gyroscope_noise_density="0.0003394"
       gyroscope_random_walk="0.000038785"
@@ -39,11 +56,5 @@
       accelerometer_turn_on_bias_sigma="0.1960"
       orientation_noise="0.01"
-      enable_local_ned_frame="false"
-      reference_frame="world"
-      update_rate="50">
-      <inertia ixx="0.00001" ixy="0.0" ixz="0.0" iyy="0.00001" iyz="0.0" izz="0.00001" />
-      <xacro:insert_block name="origin" />
-    </xacro:imu_plugin_macro>
-  </xacro:macro>
+      -->
   <xacro:macro name="default_imu_macro" params="namespace parent_link *origin inertial_reference_frame">
     <!-- ADIS16448 IMU. -->
@@ -71,13 +82,13 @@
       imu_topic="imu"
       mass_imu_sensor="0.0000015"
-      gyroscope_noise_density="0.0003394"
-      gyroscope_random_walk="0.000038785"
-      gyroscope_bias_correlation_time="1000.0"
+      gyroscope_noise_density="0.000003394"
+      gyroscope_random_walk="0.00000038785"
+      gyroscope_bias_correlation_time="100.0"
       gyroscope_turn_on_bias_sigma="0.0087"
-      accelerometer_noise_density="0.004"
-      accelerometer_random_walk="0.006"
-      accelerometer_bias_correlation_time="300.0"
+      accelerometer_noise_density="0.00004"
+      accelerometer_random_walk="0.00006"
+      accelerometer_bias_correlation_time="100.0"
       accelerometer_turn_on_bias_sigma="0.1960"
-      orientation_noise="0.01"
+      orientation_noise="0.00001"
       enable_local_ned_frame="false"
       reference_frame="world"
@@ -95,13 +106,13 @@
       imu_topic="imu2"
       mass_imu_sensor="0.015"
-      gyroscope_noise_density="0.0003394"
-      gyroscope_random_walk="0.000038785"
-      gyroscope_bias_correlation_time="1000.0"
+      gyroscope_noise_density="0.000003394"
+      gyroscope_random_walk="0.00000038785"
+      gyroscope_bias_correlation_time="100.0"
       gyroscope_turn_on_bias_sigma="0.0087"
-      accelerometer_noise_density="0.004"
-      accelerometer_random_walk="0.006"
-      accelerometer_bias_correlation_time="300.0"
+      accelerometer_noise_density="0.00004"
+      accelerometer_random_walk="0.00006"
+      accelerometer_bias_correlation_time="100.0"
       accelerometer_turn_on_bias_sigma="0.1960"
-      orientation_noise="0.01"
+      orientation_noise="0.00001"
       enable_local_ned_frame="true"
       reference_frame="world_ned"

File: uuv_sensor_plugins/uuv_sensor_ros_plugins/urdf/pose_3d_snippets.xacro (robot description, xacro)
@@ -63,5 +63,5 @@
       namespace="${namespace}"
       parent_link="${parent_link}"
-      topic="pose_gt"
+      topic="cheater"
       update_rate="20"
       noise_sigma="0.0"

File: uuv_sensor_plugins/uuv_sensor_ros_plugins/urdf/sensor_snippets.xacro (robot description, xacro)
@@ -24,3 +24,4 @@
   <xacro:include filename="$(find uuv_sensor_ros_plugins)/urdf/pose_3d_snippets.xacro" />
   <xacro:include filename="$(find uuv_sensor_ros_plugins)/urdf/chemical_concentration_snippets.xacro"/>
+  <xacro:include filename="$(find task_allocation_ros)/urdf/light_snippets.xacro"/>
 </robot>
